File: Power Switch/switch_v4.sch (EAGLE design)
At the start: 27 parts, among them U2 ATTINY10-TS8R

Commit message: updates
Parts:
- R2: value 330 -> 100
Changed lines of the file:
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@@
 <part name="C1" library="rcl" library_urn="urn:adsk.eagle:library:334" deviceset="C-EU" device="C0603K" package3d_urn="urn:adsk.eagle:package:23680/2" value="10uF"/>
 <part name="IRLML6402" library="transistor-power" library_urn="urn:adsk.eagle:library:400" deviceset="FDN360P" device="" package3d_urn="urn:adsk.eagle:package:29529/2"/>
-<part name="R2" library="rcl" library_urn="urn:adsk.eagle:library:334" deviceset="R-EU_" device="R0603" package3d_urn="urn:adsk.eagle:package:23555/2" value="330"/>
+<part name="R2" library="rcl" library_urn="urn:adsk.eagle:library:334" deviceset="R-EU_" device="R0603" package3d_urn="urn:adsk.eagle:package:23555/2" value="100"/>
 <part name="D2" library="SparkFun-LED" library_urn="urn:adsk.eagle:library:529" deviceset="LED" device="0603" package3d_urn="urn:adsk.eagle:package:39354/1"/>
 <part name="GND3" library="SparkFun-PowerSymbols" library_urn="urn:adsk.eagle:library:530" deviceset="GND" device=""/>

Commit message: PCB updates (jumper distance) and a new RGB mini board
Parts:
- removed INV, INV1: PWM INV JUMPER, SparkFun-Jumpers:JUMPER-SMT_2_NO_NO-SILK
- added JP2: JUMPER-SMT_3_NO_NO-SILK, SparkFun-Jumpers:JUMPER-SMT_3_NO_NO-SILK
- added JP3: JUMPER-SMT_2_NO_NO-SILK, SparkFun-Jumpers:JUMPER-SMT_2_NO_NO-SILK
- JP1: value JUMPER-SMT_3_2-NC_PASTE_NO-SILK -> JUMPER-SMT_2_NO_NO-SILK; device SparkFun-Jumpers:JUMPER-SMT_3_2-NC_PASTE_NO-SILK -> SparkFun-Jumpers:JUMPER-SMT_2_NO_NO-SILK
Connections:
- net 5V: now also JP1.2; no longer INV1.2
- net GND: now also JP3.1; no longer INV.1
- net IN: now also JP2.2; no longer JP1.2
- net INV: now also JP3.2; no longer INV.2
- net REG_OUT: now also JP2.3; no longer JP1.3
- net VCC: now also JP2.1; no longer INV1.1
Changed lines of the file:
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@@
 <part name="R3" library="rcl" library_urn="urn:adsk.eagle:library:334" deviceset="R-EU_" device="R0603" package3d_urn="urn:adsk.eagle:package:23555/2" value="10k"/>
 <part name="NPN" library="SparkFun-DiscreteSemi" library_urn="urn:adsk.eagle:library:514" deviceset="TRANS_NPN" device="-MMBT2222AL" package3d_urn="urn:adsk.eagle:package:38446/1" value="BC848"/>
-<part name="GND9" library="SparkFun-PowerSymbols" library_urn="urn:adsk.eagle:library:530" deviceset="GND" device=""/>
-<part name="INV" library="SparkFun-Jumpers" library_urn="urn:adsk.eagle:library:528" deviceset="JUMPER-SMT_2_NO" device="_NO-SILK" package3d_urn="urn:adsk.eagle:package:39277/1" value="PWM INV JUMPER"/>
 <part name="S1" library="SparkFun-Switches" library_urn="urn:adsk.eagle:library:535" deviceset="MOMENTARY-SWITCH-SPST" device="-SMD-4.6X2.8MM" package3d_urn="urn:adsk.eagle:package:40176/1" value="BUTTON"/>
 <part name="GND7" library="SparkFun-PowerSymbols" library_urn="urn:adsk.eagle:library:530" deviceset="GND" device=""/>
 <part name="DIN" library="testpad" library_urn="urn:adsk.eagle:library:385" deviceset="TP" device="TP15R" package3d_urn="urn:adsk.eagle:package:27968/1" value="TPTP15R"/>
 <part name="D3" library="diode" library_urn="urn:adsk.eagle:library:210" deviceset="BAT60J" device="" package3d_urn="urn:adsk.eagle:package:43461/1" value="NSR0320MW2T1G"/>
-<part name="JP1" library="SparkFun-Jumpers" library_urn="urn:adsk.eagle:library:528" deviceset="JUMPER-SMT_3_2-NC_PASTE" device="_NO-SILK" package3d_urn="urn:adsk.eagle:package:39292/1" value="JUMPER-SMT_3_2-NC_PASTE_NO-SILK"/>
-<part name="INV1" library="SparkFun-Jumpers" library_urn="urn:adsk.eagle:library:528" deviceset="JUMPER-SMT_2_NO" device="_NO-SILK" package3d_urn="urn:adsk.eagle:package:39277/1" value="PWM INV JUMPER"/>
 <part name="OUT" library="testpad" library_urn="urn:adsk.eagle:library:385" deviceset="TP" device="TP15R" package3d_urn="urn:adsk.eagle:package:27968/1" value="TPTP15R"/>
 <part name="G2" library="testpad" library_urn="urn:adsk.eagle:library:385" deviceset="TP" device="TP15R" package3d_urn="urn:adsk.eagle:package:27968/1" value="TPTP15R"/>
@@
 <part name="R5" library="rcl" library_urn="urn:adsk.eagle:library:334" deviceset="R-EU_" device="R0603" package3d_urn="urn:adsk.eagle:package:23555/2" value="1k"/>
 <part name="U2" library="ATTINY10-TS8R" deviceset="ATTINY10-TS8R" device=""/>
+<part name="JP2" library="SparkFun-Jumpers" deviceset="JUMPER-SMT_3_NO" device="_NO-SILK" package3d_urn="urn:adsk.eagle:package:39284/1"/>
+<part name="JP1" library="SparkFun-Jumpers" deviceset="JUMPER-SMT_2_NO" device="_NO-SILK" package3d_urn="urn:adsk.eagle:package:39277/1"/>
+<part name="JP3" library="SparkFun-Jumpers" deviceset="JUMPER-SMT_2_NO" device="_NO-SILK" package3d_urn="urn:adsk.eagle:package:39277/1"/>
+<part name="GND11" library="SparkFun-PowerSymbols" library_urn="urn:adsk.eagle:library:530" deviceset="GND" device=""/>
 </parts>
 <sheets>
@@
 <attribute name="VALUE" x="111.76" y="20.574" size="1.778" layer="96" font="vector"/>
 </instance>
-<instance part="GND9" gate="1" x="116.84" y="60.96" smashed="yes">
-<attribute name="VALUE" x="116.84" y="60.706" size="1.778" layer="96" align="top-center"/>
-</instance>
-<instance part="INV" gate="G$1" x="116.84" y="78.74" smashed="yes" rot="R90">
-<attribute name="NAME" x="114.3" y="76.2" size="1.778" layer="95" font="vector" rot="R90"/>
-<attribute name="VALUE" x="119.38" y="73.66" size="1.778" layer="96" font="vector" rot="R90" align="top-left"/>
-</instance>
 <instance part="S1" gate="G$1" x="160.02" y="60.96" smashed="yes">
 <attribute name="NAME" x="160.02" y="62.484" size="1.778" layer="95" font="vector" align="bottom-center"/>
@@
 <attribute name="VALUE" x="160.274" y="19.431" size="1.778" layer="96"/>
 </instance>
-<instance part="JP1" gate="G$1" x="-17.78" y="119.38" smashed="yes" rot="R90">
-<attribute name="NAME" x="-18.161" y="121.92" size="1.778" layer="95" font="vector" rot="R90"/>
-<attribute name="VALUE" x="-17.399" y="121.92" size="1.778" layer="96" font="vector" rot="R90" align="top-left"/>
-</instance>
-<instance part="INV1" gate="G$1" x="-48.26" y="12.7" smashed="yes" rot="R90">
-<attribute name="NAME" x="-50.8" y="10.16" size="1.778" layer="95" font="vector" rot="R90"/>
-<attribute name="VALUE" x="-45.72" y="7.62" size="1.778" layer="96" font="vector" rot="R90" align="top-left"/>
-</instance>
 <instance part="OUT" gate="G$1" x="-81.28" y="86.36" smashed="yes">
 <attribute name="NAME" x="-82.55" y="87.63" size="1.778" layer="95"/>
@@
 <attribute name="NAME" x="44.91655" y="121.482390625" size="2.0885" layer="95" ratio="10" rot="SR0"/>
 <attribute name="VALUE" x="37.81796875" y="98.4387" size="2.08421875" layer="96" ratio="10" rot="SR0"/>
+</instance>
+<instance part="JP2" gate="G$1" x="-50.8" y="119.38" smashed="yes" rot="R90">
+<attribute name="NAME" x="-51.181" y="121.92" size="1.778" layer="95" font="vector" rot="R90"/>
+<attribute name="VALUE" x="-50.419" y="121.92" size="1.778" layer="96" font="vector" rot="R90" align="top-left"/>
+</instance>
+<instance part="JP1" gate="G$1" x="-60.96" y="10.16" smashed="yes" rot="R90">
+<attribute name="NAME" x="-63.5" y="7.62" size="1.778" layer="95" font="vector" rot="R90"/>
+</instance>
+<instance part="JP3" gate="G$1" x="127" y="78.74" smashed="yes" rot="R90">
+<attribute name="NAME" x="124.46" y="76.2" size="1.778" layer="95" font="vector" rot="R90"/>
+</instance>
+<instance part="GND11" gate="1" x="127" y="58.42" smashed="yes">
+<attribute name="VALUE" x="127" y="58.166" size="1.778" layer="96" align="top-center"/>
 </instance>
 </instances>
@@
 </segment>
 <segment>
-<pinref part="INV1" gate="G$1" pin="2"/>
-<wire x1="-48.26" y1="17.78" x2="-48.26" y2="22.86" width="0.1524" layer="91"/>
-<wire x1="-48.26" y1="22.86" x2="-53.34" y2="22.86" width="0.1524" layer="91"/>
-<label x="-53.34" y="22.86" size="1.778" layer="95"/>
-</segment>
-<segment>
 <pinref part="U2" gate="A" pin="VCC"/>
 <label x="22.86" y="114.3" size="1.778" layer="95"/>
 <wire x1="33.02" y1="114.3" x2="22.86" y2="114.3" width="0.1524" layer="91"/>
+</segment>
+<segment>
+<pinref part="JP1" gate="G$1" pin="2"/>
+<wire x1="-60.96" y1="15.24" x2="-60.96" y2="20.32" width="0.1524" layer="91"/>
+<label x="-60.96" y="20.32" size="1.778" layer="95" rot="R90"/>
 </segment>
 </net>
@@
 <pinref part="NPN" gate="G$1" pin="E"/>
 <wire x1="111.76" y1="17.78" x2="111.76" y2="7.62" width="0.1524" layer="91"/>
-</segment>
-<segment>
-<pinref part="GND9" gate="1" pin="GND"/>
-<wire x1="116.84" y1="63.5" x2="116.84" y2="73.66" width="0.1524" layer="91"/>
-<pinref part="INV" gate="G$1" pin="1"/>
 </segment>
 <segment>
@@
 <label x="22.86" y="96.52" size="1.778" layer="95"/>
 </segment>
+<segment>
+<pinref part="JP3" gate="G$1" pin="1"/>
+<wire x1="127" y1="73.66" x2="127" y2="60.96" width="0.1524" layer="91"/>
+<pinref part="GND11" gate="1" pin="GND"/>
+</segment>
 </net>
 <net name="N$3" class="0">
@@
 </segment>
 <segment>
-<pinref part="JP1" gate="G$1" pin="1"/>
-<wire x1="-22.86" y1="119.38" x2="-30.48" y2="119.38" width="0.1524" layer="91"/>
-<label x="-33.02" y="119.38" size="1.778" layer="95"/>
-</segment>
-<segment>
-<pinref part="INV1" gate="G$1" pin="1"/>
-<wire x1="-48.26" y1="7.62" x2="-48.26" y2="-2.54" width="0.1524" layer="91"/>
-<label x="-48.26" y="-2.54" size="1.778" layer="95"/>
-</segment>
-<segment>
 <pinref part="IN" gate="G$1" pin="TP"/>
 <wire x1="-81.28" y1="58.42" x2="-81.28" y2="50.8" width="0.1524" layer="91"/>
 <label x="-81.28" y="50.8" size="1.778" layer="95" rot="R180" xref="yes"/>
+</segment>
+<segment>
+<pinref part="JP2" gate="G$1" pin="1"/>
+<wire x1="-55.88" y1="119.38" x2="-60.96" y2="119.38" width="0.1524" layer="91"/>
+<label x="-60.96" y="119.38" size="1.778" layer="95" rot="R270"/>
+</segment>
+<segment>
+<pinref part="JP1" gate="G$1" pin="1"/>
+<wire x1="-60.96" y1="5.08" x2="-60.96" y2="0" width="0.1524" layer="91"/>
+<label x="-60.96" y="0" size="1.778" layer="95" rot="R270"/>
 </segment>
 </net>
@@
 </segment>
 <segment>
-<pinref part="JP1" gate="G$1" pin="3"/>
-<wire x1="-12.7" y1="119.38" x2="-2.54" y2="119.38" width="0.1524" layer="91"/>
-<label x="-2.54" y="119.38" size="1.778" layer="95"/>
-</segment>
-<segment>
 <pinref part="OUT" gate="G$1" pin="TP"/>
 <wire x1="-81.28" y1="83.82" x2="-81.28" y2="76.2" width="0.1524" layer="91"/>
 <label x="-81.28" y="76.2" size="1.778" layer="95" rot="R180" xref="yes"/>
+</segment>
+<segment>
+<pinref part="JP2" gate="G$1" pin="3"/>
+<wire x1="-45.72" y1="119.38" x2="-43.18" y2="119.38" width="0.1524" layer="91"/>
+<label x="-43.18" y="119.38" size="1.778" layer="95" rot="R270"/>
 </segment>
 </net>
@@
 </segment>
 <segment>
-<pinref part="JP1" gate="G$1" pin="2"/>
-<wire x1="-17.78" y1="114.3" x2="-17.78" y2="109.22" width="0.1524" layer="91"/>
-<label x="-17.78" y="106.68" size="1.778" layer="95"/>
+<pinref part="JP2" gate="G$1" pin="2"/>
+<wire x1="-50.8" y1="114.3" x2="-50.8" y2="111.76" width="0.1524" layer="91"/>
+<label x="-50.8" y="109.22" size="1.778" layer="95" rot="R180"/>
 </segment>
 </net>
@@
 </segment>
 <segment>
-<pinref part="INV" gate="G$1" pin="2"/>
-<wire x1="116.84" y1="83.82" x2="116.84" y2="93.98" width="0.1524" layer="91"/>
-<label x="116.84" y="93.98" size="1.778" layer="95"/>
-</segment>
-</net>
+<pinref part="JP3" gate="G$1" pin="2"/>
+<wire x1="127" y1="83.82" x2="127" y2="93.98" width="0.1524" layer="91"/>
+<label x="127" y="93.98" size="1.778" layer="95"/>
+</segment>
+</net>
