File: RGB mini/85 SOP8 v2.brd (EAGLE design)
At the start: 12.2 x 10 mm, 6 parts, among them U2 ATTINY85-15ST

Commit message: mini PCB update
Parts:
- added R1: (no value), resistor:R0603
- moved S1 0.25 mm to (25.1, 93.0)
Connections:
- new net N$1: R1.1, U2.7
- net SCK: now also R1.2; no longer U2.7
Routing:
- net LED: track 23.9 -> 25.6 mm
- net MO: track 15.9 -> 17.1 mm
Other:
- board text removed: "MODE"
