File: RGB mini/85 SOP8 v2.sch (EAGLE design)
At the start: 6 parts, among them U2 ATTINY85-15ST

Commit message: mini PCB update
Parts:
- added R1: (no value), resistor:R-EU_R0603
Connections:
- new net N$1: J2.2, R1.1
- net SCK: now also R1.2; no longer J2.2
Changed lines of the file:
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@@
 <part name="C3" library="resistor" library_urn="urn:adsk.eagle:library:348" deviceset="C-EU" device="C0603" package3d_urn="urn:adsk.eagle:package:23616/2"/>
 <part name="J2" library="SparkFun-Connectors" library_urn="urn:adsk.eagle:library:513" deviceset="CONN_03" device="1X03_NO_SILK" package3d_urn="urn:adsk.eagle:package:38076/1"/>
+<part name="R1" library="resistor" library_urn="urn:adsk.eagle:library:348" deviceset="R-EU_" device="R0603" package3d_urn="urn:adsk.eagle:package:23555/2"/>
 </parts>
 <sheets>
@@
 <attribute name="VALUE" x="-28.194" y="12.7" size="1.778" layer="96" font="vector" rot="R90"/>
 <attribute name="NAME" x="-41.148" y="12.7" size="1.778" layer="95" font="vector" rot="R90"/>
+</instance>
+<instance part="R1" gate="G$1" x="-35.56" y="55.88" smashed="yes" rot="R90">
+<attribute name="NAME" x="-37.0586" y="52.07" size="1.778" layer="95" rot="R90"/>
+<attribute name="VALUE" x="-32.258" y="52.07" size="1.778" layer="96" rot="R90"/>
 </instance>
 </instances>
@@
 <segment>
 <pinref part="U2" gate="A" pin="PB2"/>
-<wire x1="78.74" y1="27.94" x2="86.36" y2="27.94" width="0.1524" layer="91"/>
-<label x="86.36" y="27.94" size="1.778" layer="95" xref="yes"/>
+<wire x1="78.74" y1="27.94" x2="104.14" y2="27.94" width="0.1524" layer="91"/>
+<label x="104.14" y="27.94" size="1.778" layer="95" xref="yes"/>
 </segment>
 <segment>
-<pinref part="J2" gate="J$1" pin="2"/>
-<wire x1="-35.56" y1="22.86" x2="-35.56" y2="30.48" width="0.1524" layer="91"/>
-<label x="-35.56" y="30.48" size="1.778" layer="95" rot="R90" xref="yes"/>
+<pinref part="R1" gate="G$1" pin="2"/>
+<wire x1="-35.56" y1="60.96" x2="-35.56" y2="68.58" width="0.1524" layer="91"/>
+<label x="-35.56" y="68.58" size="1.778" layer="95"/>
 </segment>
 </net>
@@
 </segment>
 </net>
+<net name="N$1" class="0">
+<segment>
+<pinref part="J2" gate="J$1" pin="2"/>
+<wire x1="-35.56" y1="22.86" x2="-35.56" y2="50.8" width="0.1524" layer="91"/>
+<pinref part="R1" gate="G$1" pin="1"/>
+</segment>
+</net>
